Commit message: removed unnecessary comments

File: kiki_description/urdf/kiki_description.urdf.xacro (robot description, xacro)
@@ -1,39 +1,3 @@
-<!-- <?xml version="1.0"?> -->
 <robot xmlns:xacro="http://www.ros.org/wiki/xacro" name="kiki_robot">
-  <!-- <xacro:macro name="kiki" params="prefix"> -->
-  <!-- <?xml version="1.0" ?> -->
-<!-- <robot name="kiki_robot" xmlns:xacro="http://ros.org/wiki/xacro"> -->
-  <!-- <xacro:include filename="$(find turtlebot3_description)/urdf/common_properties.urdf"/> -->
-  <!-- Init colour -->
-  <!-- <material name="black">
-      <color rgba="0.0 0.0 0.0 1.0"/>
-  </material>
-  <material name="dark">
-    <color rgba="0.3 0.3 0.3 1.0"/>
-  </material>
-  <material name="light_black">
-    <color rgba="0.4 0.4 0.4 1.0"/>
-  </material>
-  <material name="blue">
-    <color rgba="0.0 0.0 0.8 1.0"/>
-  </material>
-  <material name="green">
-    <color rgba="0.0 0.8 0.0 1.0"/>
-  </material>
-  <material name="grey">
-    <color rgba="0.5 0.5 0.5 1.0"/>
-  </material>
-  <material name="orange">
-    <color rgba="1.0 0.4235 0.0392 1.0"/>
-  </material>
-  <material name="brown">
-    <color rgba="0.8706 0.8118 0.7647 1.0"/>
-  </material>
-  <material name="red">
-    <color rgba="0.8 0.0 0.0 1.0"/>
-  </material>
-  <material name="white">
-    <color rgba="1.0 1.0 1.0 1.0"/>
-  </material> -->
   <link name="base_footprint"/>
   <joint name="base_joint" type="fixed">
@@ -170,4 +134,3 @@
     </inertial> -->
   </link>
-  <!-- </xacro:macro> -->
 </robot>

Commit message: added the xacro macro again

File: kiki_description/urdf/kiki_description.urdf.xacro (robot description, xacro)
@@ -1,3 +1,4 @@
 <robot xmlns:xacro="http://www.ros.org/wiki/xacro" name="kiki_robot">
+  <xacro:macro name="kiki_desc_urdf" params="prefix">
   <link name="base_footprint"/>
   <joint name="base_joint" type="fixed">
@@ -134,3 +135,4 @@
     </inertial> -->
   </link>
+  </xacro:macro>
 </robot>
