Commit message: matched joint names with urdf and changed macro name

File: kiki_control/plugin/kikibot.ros2_control.xacro (robot description, xacro)
@@ -1,17 +1,17 @@
 <?xml version="1.0"?>
 <robot xmlns:xacro="http://www.ros.org/wiki/xacro">
-  <xacro:macro name="diffbot_ros2_control" params="name prefix">
+  <xacro:macro name="kiki_ros2_control" params="name prefix">
     <ros2_control name="${name}" type="system">
       <hardware>
         <plugin>kiki_diffdrive/KikiDiffDriveHardware</plugin>
-        <!-- <param name="left_wheel_name">left_wheel_joint</param>
-        <param name="right_wheel_name">right_wheel_joint</param> -->
+        <param name="left_wheel_name">wheel_left_joint</param>
+        <param name="right_wheel_name">wheel_right_joint</param>
       </hardware>
-      <joint name="${prefix}left_wheel_joint">
+      <joint name="${prefix}wheel_left_joint">
         <command_interface name="velocity"/>
         <state_interface name="position"/>
         <state_interface name="velocity"/>
       </joint>
-      <joint name="${prefix}right_wheel_joint">
+      <joint name="${prefix}wheel_right_joint">
         <command_interface name="velocity"/>
         <state_interface name="position"/>
